File: SimonSaysPCBDesign/SimonSaysPCBDesign.kicad_sch (KiCad schematic)
At the start: 36 parts, among them J1 Screw_Terminal, SW1 SW_SPST, SW2 SW_MEC_5E, SW3 SW_MEC_5E, SW4 SW_MEC_5E, SW6 SW_MEC_5E, U1 ATmega328P-P, U2 LM7805_TO220, U3 4-Pin I2C Header, Y1 16 Mhz

Commit message: Almost finished routing PCB
Parts:
- removed D1: RED, LED_THT:LED_D5.0mm, symbol Device:LED
- removed R1: 220Ω, Resistor_SMD:R_0603_1608Metric, symbol Device:R
- removed SW2, SW3, SW4, SW6: SW_MEC_5E, Button_Switch_THT:SW_PUSH_6mm_H5mm, symbol Switch:SW_MEC_5E
- added SW2, SW3, SW4, SW5: SW_Push, Button_Switch_THT:SW_PUSH_6mm_H5mm, symbol Switch:SW_Push
- LS1: footprint Connector_PinHeader_2.54mm:PinHeader_1x02_P2.54mm_Horizontal -> Connector_PinHeader_2.54mm:PinHeader_1x02_P2.54mm_Vertical
- SW1: footprint Button_Switch_SMD:SW_SPDT_PCM12 -> Button_Switch_THT:SW_PUSH_6mm_H5mm
- TTL-232R-5V1: footprint Connector_PinHeader_2.54mm:PinHeader_1x06_P2.54mm_Horizontal -> Connector_PinHeader_2.54mm:PinHeader_1x06_P2.54mm_Vertical
- U2: footprint Package_TO_SOT_THT:TO-220-3_Vertical -> Package_TO_SOT_THT:TO-220-3_Horizontal_TabDown
- U3: footprint Connector_PinHeader_2.54mm:PinHeader_1x04_P2.54mm_Horizontal -> Connector_PinHeader_2.54mm:PinHeader_1x04_P2.54mm_Vertical
- Y1: value 16 Mhz -> CLK
Connections:
- net +5V: now also SW2.2, SW3.2, SW4.2, SW5.2
- net at R6.2: now also C8.1, SW4.1
- net at R3.2: now also C7.1, SW2.1
- net at C9.1: now also R10.2, SW5.1
- net at R8.2: now also C6.1, SW3.1
- no-connect marks 0 -> 1
